Commit message: fix knee joint names

File: robots/human_description/robots/human.urdf (robot description, URDF)
Before this commit: robot human_36dof_ISB_model, 37 links, 36 joints
Joints:
- removed joint left_knee
- removed joint right_knee
- added joint left_knee_Z: type revolute, parent left_upperleg, child left_lowerleg, origin xyz=0. -0.439 0. rpy=0 -0 0, axis 0 0 -1, limit lower=0 upper=3.14159 effort=130 velocity=18.6
- added joint right_knee_Z: type revolute, parent right_upperleg, child right_lowerleg, origin xyz=0 -0.439 0 rpy=0 -0 0, axis 0 0 -1, limit lower=0 upper=3.14159 effort=130 velocity=18.6
